File: PCB/SCART_Invader.kicad_pcb (KiCad board)
At the start: 2 copper layers, 212 x 102 mm, 119 parts, among them J1 ICSP, J10 SCART-F, J11 SCART-F, J12 SCART-F, J13 Conn_01x02_Pin, J2 12V Barrel Jack, J3 RCJ-32234, J4 SCART-F, J5 SCART-F, J6 SCART-F, J7 SCART-F, J8 SCART-F, J9 SCART-F, K1 HFD4, K10 HFD4, K11 HFD4, K12 HFD4, K13 HFD4, K14 HFD4, K15 HFD4, K16 HFD4, K17 HFD4, K18 HFD4, K19 HFD4, K2 HFD4, K20 HFD4, K21 HFD4, K22 HFD4, K23 HFD4, K24 HFD4, K25 HFD4, K3 HFD4, K4 HFD4, K5 HFD4, K6 HFD4, K7 HFD4, K8 HFD4, K9 HFD4, SW1 FP_Button, U1 MIC5891, U2 CD4051B, U3 CD4051B, U4 MIC5891, U5 ATmega328P-P, U6 TSOP384xx, U7 LM7805_TO220, U8 LM1881, Y1 16 MHz

Commit message: Updates readme, adds top cover
Parts:
- J3: value RCJ-32234 -> MR-100H
Changed lines of the file:
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@@
 			)
 		)
-		(property "Value" "RCJ-32234"
+		(property "Value" "MR-100H"
 			(at 0 8.89 0)
 			(unlocked yes)
@@
 			)
 		)
-		(property "Datasheet" "https://www.mouser.co.uk/datasheet/2/1628/rcj_32xxx-3510905.pdf"
+		(property "Datasheet" ""
 			(at 0 0 0)
 			(unlocked yes)
