File: PCB/SCART_Invader.kicad_sch (KiCad schematic)
At the start: 118 parts, among them J1 ICSP, J10 SCART-F, J11 SCART-F, J12 SCART-F, J13 Conn_01x02_Pin, J2 12V Barrel Jack, J3 RCJ-32234, J4 SCART-F, J5 SCART-F, J6 SCART-F, J7 SCART-F, J8 SCART-F, J9 SCART-F, K1 HFD4, K10 HFD4, K11 HFD4, K12 HFD4, K13 HFD4, K14 HFD4, K15 HFD4, K16 HFD4, K17 HFD4, K18 HFD4, K19 HFD4, K2 HFD4, K20 HFD4, K21 HFD4, K22 HFD4, K23 HFD4, K24 HFD4, K25 HFD4, K3 HFD4, K4 HFD4, K5 HFD4, K6 HFD4, K7 HFD4, K8 HFD4, K9 HFD4, SW1 FP_Button, U1 MIC5891, U2 CD4051B, U3 CD4051B, U4 MIC5891, U5 ATmega328P-P, U6 TSOP384xx, U7 LM7805_TO220, U8 LM1881, Y1 16 MHz

Commit message: Updates readme, adds top cover
Parts:
- J3: value RCJ-32234 -> MR-100H; Supplier (none) -> https://www.ebay.co.uk/itm/160807949159
- J5: Supplier (none) -> https://www.rapidonline.com/trucomponents-202715-scart-conn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
- K1: Supplier (none) -> https://www.tme.eu/gb/details/hfd4_12/miniature-electromagn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
- U1: Supplier (none) -> https://www.mouser.co.uk/ProductDetail/Microchip-Technology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
Changed lines of the file:
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@@
 			)
 		)
+		(property "Supplier" "https://www.tme.eu/gb/details/hfd4_12/miniature-electromagnetic-relays/hongfa-relay/"
+			(at 111.76 137.16 90)
+			(effects
+				(font
+					(size 1.27 1.27)
+				)
+				(hide yes)
+			)
+		)
 		(pin "1"
 		)
@@
 			)
 		)
+		(property "Supplier" "https://www.tme.eu/gb/details/hfd4_12/miniature-electromagnetic-relays/hongfa-relay/"
+			(at 111.76 147.32 90)
+			(effects
+				(font
+					(size 1.27 1.27)
+				)
+				(hide yes)
+			)
+		)
 		(pin "1"
 		)
@@
 			)
 		)
-		(property "Datasheet" " ~"
+		(property "Datasheet" "~"
 			(at 50.8 339.09 0)
 			(effects
@@
 			)
 		)
+		(property "Supplier" "https://www.rapidonline.com/trucomponents-202715-scart-connector-socket-right-angle-black-20-2715"
+			(at 50.8 340.36 0)
+			(effects
+				(font
+					(size 1.27 1.27)
+				)
+				(hide yes)
+			)
+		)
 		(pin "3"
 		)
@@
 			)
 		)
-		(property "Value" "RCJ-32234"
+		(property "Value" "MR-100H"
 			(at 422.402 210.82 0)
 			(effects
@@
 			)
 		)
-		(property "Datasheet" "https://www.mouser.co.uk/datasheet/2/1628/rcj_32xxx-3510905.pdf"
+		(property "Datasheet" ""
 			(at 423.926 203.454 0)
 			(effects
@@
 			)
 		)
+		(property "Supplier" "https://www.ebay.co.uk/itm/160807949159"
+			(at 422.91 217.17 0)
+			(effects
+				(font
+					(size 1.27 1.27)
+				)
+				(hide yes)
+			)
+		)
 		(pin "2"
 		)
@@
 			)
 		)
+		(property "Supplier" "https://www.mouser.co.uk/ProductDetail/Microchip-Technology/MIC5891YN?qs=kh6iOki%2FeLE0VkU6OGtmGA%3D%3D"
+			(at 359.41 43.18 0)
+			(effects
+				(font
+					(size 1.27 1.27)
+				)
+				(hide yes)
+			)
+		)
 		(pin "4"
 		)
@@
 			(effects
 				(font
+					(size 1.27 1.27)
+				)
+				(hide yes)
+			)
+		)
+		(property "Supplier" "https://www.tme.eu/gb/details/hfd4_12/miniature-electromagnetic-relays/hongfa-relay/"
+			(at 529.59 43.18 90)
+			(effects
+				(font
